File: ExternalFloppyAdapter.kicad_sch (KiCad schematic)
At the start: 22 parts, among them J1 Screw_Terminal_01x04, U3 74LS38, U4 74LS74

Commit message: Layout reworked
Connections:
- net ~{SEL1}: now reaches U_AMIGA1.21 (~{SEL1})
- net ~{SEL1}: now also J_DRIVE1.5 (Pin_5); no longer J_DRIVE1.1 (Pin_1)
- net ~{SEL2}: now reaches J_DRIVE1.3 (Pin_3), U_AMIGA1.9 (~{SEL2})
- net ~{SEL3}: now reaches U_AMIGA1.20 (~{SEL3})
- net ~{SEL3}: now also J_DRIVE1.1 (Pin_1); no longer J_DRIVE1.5 (Pin_5)
Other:
- note added: "Drive Select J_DRIVE ------------- 5-6 DF1 3-4 DF2 1-2 DF3"
- note removed: "Drive Select J_DRIVE ------------- 1-2 DF1 3-4 DF2 5-6 DF3"
- company: (none) -> Torsten Brischalle
Changed lines of the file:
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@@
 	(title_block
 		(title "Amiga External Floppy Adapter")
+		(rev "1.0")
+		(company "Torsten Brischalle")
 	)
 	(junction
@@
 	)
 	(junction
+		(at 106.68 81.28)
+		(diameter 0)
+		(color 0 0 0 0)
+	)
+	(junction
 		(at 184.15 44.45)
 		(diameter 0)
@@
 	)
 	(junction
-		(at 106.68 81.28)
-		(diameter 0)
-		(color 0 0 0 0)
-	)
-	(junction
 		(at 265.43 68.58)
 		(diameter 0)
@@
 	(wire
 		(pts
-			(xy 104.14 81.28) (xy 106.68 81.28)
+			(xy 242.57 129.54) (xy 245.11 129.54)
 		)
 		(stroke
@@
 	(wire
 		(pts
-			(xy 242.57 129.54) (xy 245.11 129.54)
+			(xy 38.1 186.69) (xy 48.26 186.69)
 		)
 		(stroke
@@
 	(wire
 		(pts
-			(xy 38.1 186.69) (xy 48.26 186.69)
+			(xy 48.26 81.28) (xy 91.44 81.28)
 		)
 		(stroke
@@
 	(wire
 		(pts
+			(xy 106.68 81.28) (xy 106.68 83.82)
+		)
+		(stroke
+			(width 0)
+			(type default)
+		)
+	)
+	(wire
+		(pts
 			(xy 133.35 49.53) (xy 137.16 49.53)
 		)
@@
 	(wire
 		(pts
+			(xy 48.26 78.74) (xy 91.44 78.74)
+		)
+		(stroke
+			(width 0)
+			(type default)
+		)
+	)
+	(wire
+		(pts
 			(xy 116.84 78.74) (xy 198.12 78.74)
 		)
@@
 	(wire
 		(pts
+			(xy 48.26 83.82) (xy 91.44 83.82)
+		)
+		(stroke
+			(width 0)
+			(type default)
+		)
+	)
+	(wire
+		(pts
 			(xy 48.26 114.3) (xy 77.47 114.3)
 		)
@@
 		)
 	)
+	(wire
+		(pts
+			(xy 104.14 81.28) (xy 106.68 81.28)
+		)
+		(stroke
+			(width 0)
+			(type default)
+		)
+	)
 	(bus
 		(pts
@@
 	(wire
 		(pts
-			(xy 48.26 83.82) (xy 91.44 83.82)
-		)
-		(stroke
-			(width 0)
-			(type default)
-		)
-	)
-	(wire
-		(pts
 			(xy 184.15 44.45) (xy 184.15 43.18)
 		)
@@
 	(wire
 		(pts
-			(xy 48.26 78.74) (xy 91.44 78.74)
-		)
-		(stroke
-			(width 0)
-			(type default)
-		)
-	)
-	(wire
-		(pts
 			(xy 48.26 168.91) (xy 38.1 168.91)
 		)
@@
 	(wire
 		(pts
-			(xy 35.56 137.16) (xy 35.56 138.43)
+			(xy 104.14 78.74) (xy 106.68 78.74)
 		)
 		(stroke
@@
 	(wire
 		(pts
-			(xy 265.43 71.12) (xy 265.43 73.66)
+			(xy 35.56 137.16) (xy 35.56 138.43)
 		)
 		(stroke
@@
 	(wire
 		(pts
-			(xy 48.26 91.44) (xy 50.8 91.44)
+			(xy 265.43 71.12) (xy 265.43 73.66)
 		)
 		(stroke
@@
 	(wire
 		(pts
-			(xy 48.26 116.84) (xy 77.47 116.84)
+			(xy 48.26 91.44) (xy 50.8 91.44)
 		)
 		(stroke
@@
 	(wire
 		(pts
-			(xy 55.88 180.34) (xy 58.42 180.34)
+			(xy 48.26 116.84) (xy 77.47 116.84)
 		)
 		(stroke
@@
 	(wire
 		(pts
-			(xy 38.1 185.42) (xy 38.1 186.69)
+			(xy 55.88 180.34) (xy 58.42 180.34)
 		)
 		(stroke
@@
 	(wire
 		(pts
-			(xy 106.68 83.82) (xy 104.14 83.82)
+			(xy 38.1 185.42) (xy 38.1 186.69)
 		)
 		(stroke
@@
 	(wire
 		(pts
-			(xy 262.89 81.28) (xy 265.43 81.28)
+			(xy 104.14 83.82) (xy 106.68 83.82)
 		)
 		(stroke
@@
 	(wire
 		(pts
-			(xy 236.22 81.28) (xy 236.22 66.04)
+			(xy 262.89 81.28) (xy 265.43 81.28)
 		)
 		(stroke
@@
 	(wire
 		(pts
-			(xy 137.16 40.64) (xy 137.16 49.53)
+			(xy 236.22 81.28) (xy 236.22 66.04)
 		)
 		(stroke
@@
 	(wire
 		(pts
-			(xy 154.94 57.15) (xy 154.94 58.42)
+			(xy 137.16 40.64) (xy 137.16 49.53)
 		)
 		(stroke
@@
 	(wire
 		(pts
-			(xy 104.14 78.74) (xy 106.68 78.74)
+			(xy 154.94 57.15) (xy 154.94 58.42)
 		)
 		(stroke
@@
 		)
 	)
-	(wire
-		(pts
-			(xy 106.68 81.28) (xy 106.68 83.82)
-		)
-		(stroke
-			(width 0)
-			(type default)
-		)
-	)
 	(bus
 		(pts
@@
 	(wire
 		(pts
-			(xy 48.26 81.28) (xy 91.44 81.28)
-		)
-		(stroke
-			(width 0)
-			(type default)
-		)
-	)
-	(wire
-		(pts
 			(xy 106.68 78.74) (xy 106.68 81.28)
 		)
@@
 		)
 	)
-	(text "Drive Select J_DRIVE\n-------------\n1-2		DF1\n3-4		DF2\n5-6		DF3"
+	(text "Drive Select J_DRIVE\n-------------\n5-6		DF1\n3-4		DF2\n1-2		DF3"
 		(exclude_from_sim no)
 		(at 95.25 99.06 0)
@@
 		)
 	)
+	(label "~{SEL3}"
+		(at 50.8 83.82 0)
+		(effects
+			(font
+				(size 1.27 1.27)
+			)
+			(justify left bottom)
+		)
+	)
 	(label "~{INDEX}"
 		(at 68.58 73.66 0)
@@
 		)
 	)
+	(label "~{SEL1}"
+		(at 50.8 78.74 0)
+		(effects
+			(font
+				(size 1.27 1.27)
+			)
+			(justify left bottom)
+		)
+	)
 	(label "~{CHNG}"
 		(at 50.8 71.12 0)
@@
 		)
 	)
+	(label "~{SEL2}"
+		(at 50.8 81.28 0)
+		(effects
+			(font
+				(size 1.27 1.27)
+			)
+			(justify left bottom)
+		)
+	)
 	(label "~{DIR}"
 		(at 68.58 88.9 0)
@@
 		(lib_id "Connector_Generic:Conn_02x03_Odd_Even")
 		(at 96.52 81.28 0)
+		(mirror x)
 		(unit 1)
 		(exclude_from_sim no)
@@
 		(on_board yes)
 		(dnp no)
-		(fields_autoplaced yes)
 		(property "Reference" "J_DRIVE1"
 			(at 97.79 72.39 0)

Commit message: Floppy connector changed, layout improved
Parts:
- U_AMIGA1: footprint Amiga500:ExternalFloppyConnector -> Amiga500:ExternalFloppyConnectorEdgeMount
Changed lines of the file:
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@@
 			)
 		)
-		(property "Footprint" "Amiga500:ExternalFloppyConnector"
+		(property "Footprint" "Amiga500:ExternalFloppyConnectorEdgeMount"
 			(at 35.56 91.44 0)
 			(effects
